File: Power.kicad_sch (KiCad schematic)
At the start: 42 parts, among them J1 XT60_BAT, J102 E_STOP, Q1 SQJ459EP-T1_GE3, U1 LMR36520FADDA, U2 AP2112K-3.3

Commit message: Finalize Rev 1.1d robustness, thermal layout and manufacturing package
Preserve sensing and current-limit fixes, assembly part/rotation corrections,
D2 package changes, revision markings and incremental thermal copper/vias.
Archive the working checkpoints and supplier/validation evidence alongside
matched Gerbers, BOM, CPL, schematic PDF, renders and hash manifests.

Current Rev 1.1d: ERC 0; DRC 0 errors, 0 opens and 0 parity issues,
with 19 existing library footprint warnings. Preserve original routing and
component placements; physical powered qualification is not yet performed.
Relay alignment requires assembler review before assembly.
Parts:
- D2: value SMCJ30A -> TVS3300DRVR; footprint Diode_SMD:D_SMC -> abx-footprints:TVS3300_DRV0006A_2x2mm; symbol Device:D_TVS -> abx:TVS3300DRVR
- R2: value 100k -> 150k
- R6: value 10k -> 22k
Connections:
- net +BATT: now also D2.4 (IN), D2.5 (IN), D2.6 (IN); no longer D2.1 (A1)
- net GND: now also D2.1 (GND), D2.3 (GND), D2.7 (EP_GND)
Other:
- note added: "D2: 33V standoff; 40V max at specified 8/20us pulse. No continuous braking-energy rating."
- title: (none) -> ABX-Motion
