File: Industrial_IO.kicad_sch (KiCad schematic)
At the start: 43 parts, among them J601 B3B-PH-K-S, J602 B3B-PH-K-S, J603 B3B-PH-K-S, J604 B3B-PH-K-S, J605 B3B-PH-K-S, J606 B3B-PH-K-S, Q601 AO3400A, Q602 AO3400A, U601 PCA9555PW,118

Commit message: Finalize V1.1 rear exposed-copper gold gear branding, polish, validation, and production package
Parts:
- F5: value 500mA_PTC -> 1206L050/15YR
Changed lines of the file:
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@@
 			)
 		)
-		(property "Value" "500mA_PTC"
+		(property "Value" "1206L050/15YR"
 			(at 284.48 44.45 0)
 			(effects

Commit message: Finalize Rev 1.1d robustness, thermal layout and manufacturing package
Preserve sensing and current-limit fixes, assembly part/rotation corrections,
D2 package changes, revision markings and incremental thermal copper/vias.
Archive the working checkpoints and supplier/validation evidence alongside
matched Gerbers, BOM, CPL, schematic PDF, renders and hash manifests.

Current Rev 1.1d: ERC 0; DRC 0 errors, 0 opens and 0 parity issues,
with 19 existing library footprint warnings. Preserve original routing and
component placements; physical powered qualification is not yet performed.
Relay alignment requires assembler review before assembly.
Other:
- title: (none) -> ABX-Motion
Changed lines of the file:
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@@
 	(generator_version "10.0")
 	(paper "A3")
+	(title_block (title "ABX-Motion") (rev "1.1d"))
 	(text "SHEET 5: 6x 3-PIN JST-PH INDUSTRIAL I/O (8x LIMIT/GPIO + 2x 5V/500mA DC OUTPUTS) & PCA9555PW EXPANDER"
 		(exclude_from_sim no)

Commit message: Save Rev 1.2a three-axis checkpoint and audited JLCPCB exports
Parts:
- removed R621, R622: 10k, Resistor_SMD:R_0603_1608Metric, symbol Device:R
- added C610, C611, C612, C613: 10nF, Capacitor_SMD:C_0603_1608Metric, symbol Device:C
- added J607, J608: B3B-PH-K-S, Connector_JST:JST_PH_B3B-PH-K_1x03_P2.00mm_Vertical, symbol Connector:Conn_01x03_Pin
- added R623, R624, R627, R628: 4.7k, Resistor_SMD:R_0603_1608Metric, symbol Device:R
- added R625, R626, R629, R630: 1k, Resistor_SMD:R_0603_1608Metric, symbol Device:R
- C601: LCSC (none) -> C14663
- C602, C603, C604, C605, C606, C607, C608, C609: LCSC (none) -> C57112
- D601, D602: LCSC (none) -> C8598
- F5: LCSC (none) -> C151162
- J601, J602, J603, J604, J605, J606: LCSC (none) -> C131339
- Q601, Q602: LCSC (none) -> C20917
- R601, R602, R603, R604, R605, R606, R607, R608: LCSC (none) -> C23162
- R609, R610, R611, R612, R613, R614, R615, R616, R617, R618: LCSC (none) -> C21190
- R619, R620: LCSC (none) -> C22775
- U601: LCSC (none) -> C128392
Connections:
- net +3V3: now also R623.1, R624.1, R627.1, R628.1
- net GND: now also C610.2, C611.2, C612.2, C613.2, J607.2 (Pin_2), J608.2 (Pin_2)
- net S1_MAX_IN renamed X_MAX_IN
- net S1_MAX_RAW renamed X_MAX_RAW
- net S1_MIN_IN renamed X_MIN_IN
- net S1_MIN_RAW renamed X_MIN_RAW
- net S2_MAX_IN renamed Y_MAX_IN
- net S2_MAX_RAW renamed Y_MAX_RAW
- net S2_MIN_IN renamed Y_MIN_IN
- net S2_MIN_RAW renamed Y_MIN_RAW
- net STEP1_EN renamed DIN1_IN
- net DIN1_IN: now also C612.1, R629.2
- net STEP2_EN renamed DIN2_IN
- net DIN2_IN: now also C613.1, R630.2
- new net DIN1_RAW: J608.1 (Pin_1), R627.2, R629.1
- new net DIN2_RAW: J608.3 (Pin_3), R628.2, R630.1
- new net Z_MAX_IN: C611.1, R626.2
- new net Z_MAX_RAW: J607.3 (Pin_3), R624.2, R626.1
- new net Z_MIN_IN: C610.1, R625.2
- new net Z_MIN_RAW: J607.1 (Pin_1), R623.2, R625.1
Other:
- note added: "3V3 / DRY CONTACT ONLY"
- note added: "DIN: U601 IO1_2 / IO1_3"
- note added: "SPARE INPUTS: DIN1 / GND / DIN2"
- note added: "Z LIMITS: MIN / GND / MAX; 3V3 / DRY CONTACT ONLY"
- note added: "Z: U704 IO1_6 / IO1_7"
- note added: "pins 15 / 16"
- note added: "pins 19 / 20"
