File: MCU.kicad_sch (KiCad schematic)
At the start: 75 parts, among them J201 USB-C, J202 ENC1_CONN, J203 ENC2_CONN, J204 CAN_TERM, J205 CAN_BUS, J206 RS485_TERM, J207 RS485_BUS, J208 OLED_I2C, J209 I2C_EXP, SW201 RESET, SW202 BOOT, SW203 BTN_BACK, SW204 BTN_NEXT, SW205 BTN_HOME, U201 USBLC6-2SC6, U202 TCAN1042V-Q1, U203 THVD1450DR, U3 ESP32-S3-WROOM-1-N8R2, U4 74LVC14A

Commit message: Release v1.0-production: finalize F1 3D STEP model alignment and archive V1.0 production package
Parts:
- removed F2, F3: 500mA_PTC, Fuse:Fuse_1206_3216Metric, symbol Device:Polyfuse
- removed F4: 250mA_PTC, Fuse:Fuse_1206_3216Metric, symbol Device:Polyfuse
- removed H5, H6: M2_OLED, MountingHole:MountingHole_2.2mm_M2, symbol Mechanical:MountingHole
- R222, R223: value 330R -> 10k
- U203: value THVD1450DR -> MAX3485
- U3: value ESP32-S3-WROOM-1-N8R2 -> ESP32-S3-WROOM-1
Connections:
- net +3V3_EXT is gone; now on net +3V3: J209.2 (Pin_2)
- net +5V_ENC is gone; now on net +5V: J202.1 (Pin_1), J203.1 (Pin_1)
- net VBUS_FUSED is gone; now on net VBUS_USB: D202.2 (A)
Other:
- moved on the sheet: U201

Commit message: Complete V1.1 compact 6-channel I/O & DC output architecture (0 ERC, 0 DRC errors, 0 unconnected, 0 parity)
Parts:
- added F2, F3: 500mA_PTC, Fuse:Fuse_1206_3216Metric, symbol Device:Polyfuse
- added F4: 250mA_PTC, Fuse:Fuse_1206_3216Metric, symbol Device:Polyfuse
- added H5, H6: M2_OLED, MountingHole:MountingHole_2.2mm_M2, symbol Mechanical:MountingHole
- R222, R223: value 10k -> 330R
- U203: value MAX3485 -> THVD1450DR
- U3: value ESP32-S3-WROOM-1 -> ESP32-S3-WROOM-1-N8R2
Connections:
- net +3V3: now also F4.1; no longer J209.2 (Pin_2)
- net +5V: now also F3.1; no longer J202.1 (Pin_1), J203.1 (Pin_1)
- net BTN_BACK: now also U3.23 (IO21); no longer U3.29 (IO36)
- net VBUS_USB: now also F2.1; no longer D202.2 (A)
- net STEP_ENABLE renamed IO_INT_N
- net IO_INT_N: now also U3.29 (IO36); no longer U3.23 (IO21)
- new net +3V3_EXT: F4.2, J209.2 (Pin_2)
- new net +5V_ENC: F3.2, J202.1 (Pin_1), J203.1 (Pin_1)
- new net VBUS_FUSED: D202.2 (A), F2.2
Other:
- moved on the sheet: U201

Commit message: Finalize Rev 1.1d robustness, thermal layout and manufacturing package
Preserve sensing and current-limit fixes, assembly part/rotation corrections,
D2 package changes, revision markings and incremental thermal copper/vias.
Archive the working checkpoints and supplier/validation evidence alongside
matched Gerbers, BOM, CPL, schematic PDF, renders and hash manifests.

Current Rev 1.1d: ERC 0; DRC 0 errors, 0 opens and 0 parity issues,
with 19 existing library footprint warnings. Preserve original routing and
component placements; physical powered qualification is not yet performed.
Relay alignment requires assembler review before assembly.
Other:
- title: (none) -> ABX-Motion
Changed lines of the file:
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@@
 	(generator_version "10.0")
 	(paper "A3")
+	(title_block (title "ABX-Motion") (rev "1.1d"))
 	(text "SHEET 2: ESP32-S3-WROOM-1, USB-C, 74LVC14A ENCODERS, CAN, RS-485, OLED & UI BUTTONS"
 		(exclude_from_sim no)

Commit message: Pack digital I/O beneath OLED and straighten local routing
Parts:
- J208: footprint Connector_PinSocket_2.54mm:PinSocket_1x04_P2.54mm_Vertical -> abx-footprints:OLED_Socket_SLW_1x04_P2.54mm_LowProfile
Changed lines of the file:
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@@
 			)
 		)
-		(property "Footprint" "Connector_PinSocket_2.54mm:PinSocket_1x04_P2.54mm_Vertical"
+		(property "Footprint" "abx-footprints:OLED_Socket_SLW_1x04_P2.54mm_LowProfile"
 			(at 314.96 215.9 0)
 			(effects
@@
 			)
 		)
-		(property "Datasheet" "~"
+		(property "Datasheet" "https://suddendocs.samtec.com/catalog_english/slw.pdf"
 			(at 314.96 215.9 0)
 			(effects

Commit message: Save Rev 1.2a three-axis checkpoint and audited JLCPCB exports
Parts:
- C201: LCSC (none) -> C15850
- C202, C203, C204, C209, C210, C211, C212, C213, C214: LCSC (none) -> C14663
- C205, C206, C207, C208: LCSC (none) -> C1588
- D201: LCSC (none) -> C78428
- D202: LCSC (none) -> C8598
- F2, F3: LCSC (none) -> C2984676
- F4: LCSC (none) -> C20798
- J201: LCSC (none) -> C165948
- J202, J203, J209: LCSC (none) -> C566014
- J204, J206: LCSC (none) -> C492401
- J205, J207: LCSC (none) -> C72334
- LED201, LED202: LCSC (none) -> C2287
- LED203: LCSC (none) -> C2288
- R201, R202: LCSC (none) -> C23186
- R203, R204, R205, R206, R207, R208, R209, R210, R227, R228, R229, R231, R232: LCSC (none) -> C25804
- R211, R213, R215, R217, R225, R226: LCSC (none) -> C23162
- R212, R214, R216, R218, R220, R224, R230: LCSC (none) -> C21190
- R219, R221: LCSC (none) -> C22787
- R222, R223: LCSC (none) -> C23138
- SW201, SW202, SW203, SW204, SW205: LCSC (none) -> C231329
- U201: LCSC (none) -> C7519
- U202: LCSC (none) -> C132550
- U203: LCSC (none) -> C2671361
- U3: LCSC (none) -> C2913204
- U4: LCSC (none) -> C133541
Connections:
- net BTN_BACK: no longer U3.23 (IO21)
- net BTN_HOME: no longer U3.33 (IO40)
- net BTN_NEXT: no longer U3.30 (IO37)
- net RELAY_1: no longer U3.24 (IO47)
- net RELAY_2: no longer U3.25 (IO48)
- net STEP_ARM: now reaches U3.26 (IO45)
- new net STEP3_DIR: U3.25 (IO48)
- new net STEP3_PUL: U3.24 (IO47)
- new net STEP_SPI_MISO: U3.33 (IO40)
- new net STEP_SPI_MOSI: U3.30 (IO37)
- new net STEP_SPI_SCLK: U3.23 (IO21)
- no-connect marks 6 -> 5

Commit message: Clear root project DRC findings and preserve explicit Ethernet draft status
Parts:
- H5: footprint MountingHole:MountingHole_2.2mm_M2 -> abx-footprints:ABX_H5_MountingHole_2.2mm_M2
- H6: footprint MountingHole:MountingHole_2.2mm_M2 -> abx-footprints:ABX_H6_MountingHole_2.2mm_M2
- J205: footprint TerminalBlock_Phoenix:TerminalBlock_Phoenix_MKDS-1,5-3-5.08_1x03_P5.08mm_Horizontal -> abx-footprints:ABX_J205_TerminalBlock_Phoenix_MKDS-1_5-3-5.08_1x03_P5.08mm_Horizontal
- J207: footprint TerminalBlock_Phoenix:TerminalBlock_Phoenix_MKDS-1,5-3-5.08_1x03_P5.08mm_Horizontal -> abx-footprints:ABX_J207_TerminalBlock_Phoenix_MKDS-1_5-3-5.08_1x03_P5.08mm_Horizontal
- U3: footprint RF_Module:ESP32-S3-WROOM-1 -> abx-footprints:ABX_U3_ESP32-S3-WROOM-1
Changed lines of the file:
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@@
 			)
 		)
-		(property "Footprint" "RF_Module:ESP32-S3-WROOM-1"
+		(property "Footprint" "abx-footprints:ABX_U3_ESP32-S3-WROOM-1"
 			(at 88.9 88.9 0)
 			(effects
@@
 			)
 		)
-		(property "Footprint" "TerminalBlock_Phoenix:TerminalBlock_Phoenix_MKDS-1,5-3-5.08_1x03_P5.08mm_Horizontal"
+		(property "Footprint" "abx-footprints:ABX_J205_TerminalBlock_Phoenix_MKDS-1_5-3-5.08_1x03_P5.08mm_Horizontal"
 			(at 119.38 218.44 0)
 			(effects
@@
 			)
 		)
-		(property "Footprint" "TerminalBlock_Phoenix:TerminalBlock_Phoenix_MKDS-1,5-3-5.08_1x03_P5.08mm_Horizontal"
+		(property "Footprint" "abx-footprints:ABX_J207_TerminalBlock_Phoenix_MKDS-1_5-3-5.08_1x03_P5.08mm_Horizontal"
 			(at 269.24 215.9 0)
 			(effects
@@
 			)
 		)
-		(property "Footprint" "MountingHole:MountingHole_2.2mm_M2"
+		(property "Footprint" "abx-footprints:ABX_H5_MountingHole_2.2mm_M2"
 			(at 347.98 185.42 0)
 			(effects
@@
 			)
 		)
-		(property "Footprint" "MountingHole:MountingHole_2.2mm_M2"
+		(property "Footprint" "abx-footprints:ABX_H6_MountingHole_2.2mm_M2"
 			(at 373.38 185.42 0)
 			(effects
