File: Steppers_Relays.kicad_sch (KiCad schematic)
At the start: 26 parts, among them J501 STEP1_MOTOR, J502 STEP1_EXT, J503 STEP2_MOTOR, J504 STEP2_EXT, J505 RELAY1_OUT, J506 RELAY2_OUT, K501 G5LE-14-DC5, K502 G5LE-14-DC5, Q501 AO3400A, Q502 AO3400A, SW501 MICROSTEP_CFG, SW502 MICROSTEP_CFG, U501 StepStick_DRV8825, U502 StepStick_DRV8825

Commit message: Complete V1.1 compact 6-channel I/O & DC output architecture (0 ERC, 0 DRC errors, 0 unconnected, 0 parity)
Parts:
- added Q503, Q504: AO3400A, Package_TO_SOT_SMD:SOT-23, symbol Transistor_FET:Q_NMOS_GSD
- added R507, R508: 10k, Resistor_SMD:R_0603_1608Metric, symbol Device:R
Connections:
- net +3V3: now also R507.1, R508.1
- net +3V3_DRV_EN: now also Q503.1 (G), Q504.1 (G)
- net STEP_ENABLE renamed STEP1_EN_GATED
- net STEP1_EN_GATED: now also Q503.3 (D), R507.2; no longer J504.1 (Pin_1), U502.9 (~{EN})
- new net STEP1_EN: Q503.2 (S)
- new net STEP2_EN: Q504.2 (S)
- new net STEP2_EN_GATED: J504.1 (Pin_1), Q504.3 (D), R508.2, U502.9 (~{EN})

Commit message: Finalize Rev 1.1d robustness, thermal layout and manufacturing package
Preserve sensing and current-limit fixes, assembly part/rotation corrections,
D2 package changes, revision markings and incremental thermal copper/vias.
Archive the working checkpoints and supplier/validation evidence alongside
matched Gerbers, BOM, CPL, schematic PDF, renders and hash manifests.

Current Rev 1.1d: ERC 0; DRC 0 errors, 0 opens and 0 parity issues,
with 19 existing library footprint warnings. Preserve original routing and
component placements; physical powered qualification is not yet performed.
Relay alignment requires assembler review before assembly.
Parts:
- U501, U502: footprint Module:Pololu_Breakout-16_15.2x20.3mm -> abx-footprints:StepStick_Socket_2x08_P2.54mm_D1.0
Other:
- title: (none) -> ABX-Motion
Changed lines of the file:
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@@
 	(generator_version "10.0")
 	(paper "A3")
+	(title_block (title "ABX-Motion") (rev "1.1d"))
 	(text "SHEET 4: DUAL STEPSTICK STEPPER CHANNELS & DUAL 5V OMRON G5LE RELAY OUTPUTS"
 		(exclude_from_sim no)
@@
 			)
 		)
-		(property "Footprint" "Module:Pololu_Breakout-16_15.2x20.3mm"
+		(property "Footprint" "abx-footprints:StepStick_Socket_2x08_P2.54mm_D1.0"
 			(at 68.58 78.74 0)
 			(effects
@@
 			)
 		)
-		(property "Footprint" "Module:Pololu_Breakout-16_15.2x20.3mm"
+		(property "Footprint" "abx-footprints:StepStick_Socket_2x08_P2.54mm_D1.0"
 			(at 215.9 78.74 0)
 			(effects

Commit message: Use low-profile EXT control headers with matching front and rear legends
Parts:
- J502, J504: footprint Connector_JST:JST_XH_B4B-XH-A_1x04_P2.50mm_Vertical -> abx-footprints:EXT_Header_1x04_P2.54mm_RightAngle; MPN (none) -> 61300411021; Manufacturer (none) -> Wurth Elektronik
Changed lines of the file:
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@@
 			)
 		)
-		(property "Footprint" "Connector_JST:JST_XH_B4B-XH-A_1x04_P2.50mm_Vertical"
+		(property "Footprint" "abx-footprints:EXT_Header_1x04_P2.54mm_RightAngle"
 			(at 114.3 111.76 0)
 			(effects
@@
 			)
 		)
-		(property "Datasheet" "~"
+		(property "Datasheet" "https://www.we-online.com/components/products/datasheet/61300411021.pdf"
 			(at 114.3 111.76 0)
 			(effects
@@
 				(hide yes)
 			)
+		)
+		(property "Manufacturer" "Wurth Elektronik"
+			(at 114.3 104.14 0)
+			(effects (font (size 1.27 1.27)) (hide yes))
+		)
+		(property "MPN" "61300411021"
+			(at 114.3 104.14 0)
+			(effects (font (size 1.27 1.27)) (hide yes))
 		)
 		(pin "1"
@@
 			)
 		)
-		(property "Footprint" "Connector_JST:JST_XH_B4B-XH-A_1x04_P2.50mm_Vertical"
+		(property "Footprint" "abx-footprints:EXT_Header_1x04_P2.54mm_RightAngle"
 			(at 261.62 111.76 0)
 			(effects
@@
 			)
 		)
-		(property "Datasheet" "~"
+		(property "Datasheet" "https://www.we-online.com/components/products/datasheet/61300411021.pdf"
 			(at 261.62 111.76 0)
 			(effects
@@
 			)
 		)
-		(pin "1"
+		(property "Manufacturer" "Wurth Elektronik"
+			(at 261.62 104.14 0)
+			(effects (font (size 1.27 1.27)) (hide yes))
+		)
+		(property "MPN" "61300411021"
+			(at 261.62 104.14 0)
+			(effects (font (size 1.27 1.27)) (hide yes))
+		)
+		(pin "1"

Commit message: Pack upright EXT headers and symmetric motor connectors to the right
Parts:
- J502, J504: footprint abx-footprints:EXT_Header_1x04_P2.54mm_RightAngle -> abx-footprints:EXT_Header_1x04_P2.54mm_Vertical; MPN 61300411021 -> 61300411121
Changed lines of the file:
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@@
 			)
 		)
-		(property "Footprint" "abx-footprints:EXT_Header_1x04_P2.54mm_RightAngle"
+		(property "Footprint" "abx-footprints:EXT_Header_1x04_P2.54mm_Vertical"
 			(at 114.3 111.76 0)
 			(effects
@@
 			)
 		)
-		(property "Datasheet" "https://www.we-online.com/components/products/datasheet/61300411021.pdf"
+		(property "Datasheet" "https://www.we-online.com/components/products/datasheet/61300411121.pdf"
 			(at 114.3 111.76 0)
 			(effects
@@
 			(effects (font (size 1.27 1.27)) (hide yes))
 		)
-		(property "MPN" "61300411021"
+		(property "MPN" "61300411121"
 			(at 114.3 104.14 0)
 			(effects (font (size 1.27 1.27)) (hide yes))
@@
 			)
 		)
-		(property "Footprint" "abx-footprints:EXT_Header_1x04_P2.54mm_RightAngle"
+		(property "Footprint" "abx-footprints:EXT_Header_1x04_P2.54mm_Vertical"
 			(at 261.62 111.76 0)
 			(effects
@@
 			)
 		)
-		(property "Datasheet" "https://www.we-online.com/components/products/datasheet/61300411021.pdf"
+		(property "Datasheet" "https://www.we-online.com/components/products/datasheet/61300411121.pdf"
 			(at 261.62 111.76 0)
 			(effects
@@
 			(effects (font (size 1.27 1.27)) (hide yes))
 		)
-		(property "MPN" "61300411021"
+		(property "MPN" "61300411121"
 			(at 261.62 104.14 0)
 			(effects (font (size 1.27 1.27)) (hide yes))

Commit message: Save Rev 1.2a three-axis checkpoint and audited JLCPCB exports
Parts:
- removed C501, C502: 100uF, Capacitor_SMD:CP_Elec_8x10.5, symbol Device:C_Polarized
- removed J501: STEP1_MOTOR, Connector_JST:JST_XH_B4B-XH-A_1x04_P2.50mm_Vertical, symbol Connector:Conn_01x04_Pin
- removed J502: STEP1_EXT, abx-footprints:EXT_Header_1x04_P2.54mm_Vertical, symbol Connector:Conn_01x04_Pin
- removed J503: STEP2_MOTOR, Connector_JST:JST_XH_B4B-XH-A_1x04_P2.50mm_Vertical, symbol Connector:Conn_01x04_Pin
- removed J504: STEP2_EXT, abx-footprints:EXT_Header_1x04_P2.54mm_Vertical, symbol Connector:Conn_01x04_Pin
- removed Q503, Q504: AO3400A, Package_TO_SOT_SMD:SOT-23, symbol Transistor_FET:Q_NMOS_GSD
- removed R505, R506, R507, R508: 10k, Resistor_SMD:R_0603_1608Metric, symbol Device:R
- removed SW501, SW502: MICROSTEP_CFG, Button_Switch_SMD:SW_DIP_SPSTx03_Slide_9.78x9.8mm_W8.61mm_P2.54mm, symbol Switch:SW_DIP_x03
- removed U501, U502: StepStick_DRV8825, abx-footprints:StepStick_Socket_2x08_P2.54mm_D1.0, symbol Driver_Motor:Pololu_Breakout_DRV8825
- added C711, C712, C721, C722, C731, C732: 10nF 63V X7R, Capacitor_SMD:C_0603_1608Metric, symbol Device:C
- added C713, C723, C733: 100nF 63V X7R, Capacitor_SMD:C_0603_1608Metric, symbol Device:C
- added C714, C724, C734: 1uF 16V X7R, Capacitor_SMD:C_0603_1608Metric, symbol Device:C
- added C715, C725, C735, C741, C742, C743, C744, C745, C746, C747, C748, C749: 100nF 16V X7R, Capacitor_SMD:C_0603_1608Metric, symbol Device:C
- added C716, C726, C736: 1uF 10V X7R, Capacitor_SMD:C_0603_1608Metric, symbol Device:C
- added C717, C727, C737: 100uF 63V, Capacitor_THT:CP_Radial_D8.0mm_P3.50mm, symbol Device:C_Polarized
- added J701, J702, J703: EXT 5V TTL EN_N STEP DIR GND, Connector_PinHeader_2.54mm:PinHeader_1x04_P2.54mm_Vertical, symbol Connector:Conn_01x04_Pin
- added J711: JST-XH MOTOR 1, Connector_JST:JST_XH_B4B-XH-A_1x04_P2.50mm_Vertical, symbol Connector:Conn_01x04_Pin
- added J712: JST-XH MOTOR 2, Connector_JST:JST_XH_B4B-XH-A_1x04_P2.50mm_Vertical, symbol Connector:Conn_01x04_Pin
- added J713: JST-XH MOTOR 3, Connector_JST:JST_XH_B4B-XH-A_1x04_P2.50mm_Vertical, symbol Connector:Conn_01x04_Pin
- added JP701, JP702, JP703: ONBOARD / EXT, Connector_PinHeader_2.54mm:PinHeader_1x03_P2.54mm_Vertical, symbol Connector:Conn_01x03_Pin
- added R711, R712, R713, R714, R715, R716, R717, R718, R721, R722, R723, R724, R725, R726, R727, R728, R731, R732, R733, R734, R735, R736, R737, R738, R744, R745, R746, R747, R748, R749, R750: 10k, Resistor_SMD:R_0603_1608Metric, symbol Device:R
- added R751, R752, R753, R754, R755, R756, R757, R758, R759: 100, Resistor_SMD:R_0603_1608Metric, symbol Device:R
- added R761, R762, R763, R764, R765: 1k, Resistor_SMD:R_0603_1608Metric, symbol Device:R
- added U701, U702, U703: DRV8462DDWR, abx-footprints:DRV8462_DDW0044E, symbol abx-r12:DRV8462DDWR
- added U704: PCA9555PW,118, Package_SO:TSSOP-24_4.4x7.8mm_P0.65mm, symbol Interface_Expansion:PCA9555PW
- added U705, U706, U707: SN74AHCT14PWR, Package_SO:TSSOP-14_4.4x5mm_P0.65mm, symbol abx-r12:SN74AHCT14PWR
- added U708, U711: SN74HC08PWR, Package_SO:TSSOP-14_4.4x5mm_P0.65mm, symbol abx-r12:SN74HC08PWR
- added U709: SN74HC74PWR, Package_SO:TSSOP-14_4.4x5mm_P0.65mm, symbol abx-r12:SN74HC74PWR
- added U710: TPS3431SDRBR, abx-footprints:TPS3431_DRB0008A, symbol abx-r12:TPS3431SDRBR
- added U712: SN74LVC2G08DCUR, Package_SO:VSSOP-8_2.3x2mm_P0.5mm, symbol abx-r12:SN74LVC2G08DCUR
- D501, D503: LCSC (none) -> C2128
- D502, D504: LCSC (none) -> C12624
- J505, J506: LCSC (none) -> C72334
- K501, K502: LCSC (none) -> C116963
- Q501, Q502: LCSC (none) -> C20917
- R501, R503: LCSC (none) -> C22775
- R502, R504: LCSC (none) -> C21190
Connections:
- net +3V3: now also C715.1, C725.1, C735.1, C741.1, C745.1, C746.1, C747.1, C748.1, C749.1, R712.1, R713.1, R714.1, R715.1, R722.1, R723.1, R724.1, R725.1, R732.1, R733.1, R734.1, R735.1, R745.1, R746.1, R750.1, U701.25 (VCC), U702.25 (VCC), U703.25 (VCC), U704.21 (A0), U704.24 (VDD), U708.14 (VCC), U709.10 (nPRE2), U709.14 (VCC), U709.2 (D1), U709.4 (nPRE1), U710.1 (VDD), U710.5 (SET1), U711.14 (VCC), U712.8 (VCC)
- net +3V3_DRV_EN: now also U708.1 (1A)
- net +5V: now also C742.1, C743.1, C744.1, U705.14 (VCC), U706.14 (VCC), U707.14 (VCC)
- net +BATT: now also C711.1, C712.1, C714.2, C717.1, C721.1, C722.1, C724.2, C727.1, C731.1, C732.1, C734.2, C737.1, U701.11 (VM), U701.12 (VM), U701.2 (VM), U701.21 (VM), U702.11 (VM), U702.12 (VM), U702.2 (VM), U702.21 (VM), U703.11 (VM), U703.12 (VM), U703.2 (VM), U703.21 (VM)
- net GND: now also C711.2, C712.2, C715.2, C716.2, C717.2, C721.2, C722.2, C725.2, C726.2, C727.2, C731.2, C732.2, C735.2, C736.2, C737.2, C741.2, C742.2, C743.2, C744.2, C745.2, C746.2, C747.2, C748.2, C749.2, J701.4 (Pin_4), J702.4 (Pin_4), J703.4 (Pin_4), R711.2, R716.2, R717.2, R718.2, R721.2, R726.2, R727.2, R728.2, R731.2, R736.2, R737.2, R738.2, R744.2, R747.2, R748.2, R749.2, R761.2, R762.2, R763.2, R764.2, R765.2, U701.10 (PGNDA), U701.13 (PGNDB), U701.20 (PGNDB), U701.22 (GND), U701.23 (GND), U701.3 (PGNDA), U701.45 (EP_GND), U702.10 (PGNDA), U702.13 (PGNDB), U702.20 (PGNDB), U702.22 (GND), U702.23 (GND), U702.3 (PGNDA), U702.45 (EP_GND), U703.10 (PGNDA), U703.13 (PGNDB), U703.20 (PGNDB), U703.22 (GND), U703.23 (GND), U703.3 (PGNDA), U703.45 (EP_GND), U704.12 (VSS), U704.2 (A1), U704.3 (A2), U705.13 (6A), U705.7 (GND), U706.13 (6A), U706.7 (GND), U707.13 (6A), U707.7 (GND), U708.7 (GND), U709.11 (CLK2), U709.12 (D2), U709.13 (nCLR2), U709.7 (GND), U710.4 (GND), U710.9 (EP_GND), U711.7 (GND), U712.4 (GND)
- net RELAY_1: now also U712.7 (1Y)
- net RELAY_2: now also U712.3 (2Y)
- net STEP1_DIR: now also R718.1, U701.40 (DIR), U705.5 (3A)
- net STEP1_PUL: now also R717.1, U701.39 (STEP), U705.1 (1A)
- net STEP2_DIR: now also R728.1, U702.40 (DIR), U706.5 (3A)
- net STEP2_PUL: now also R727.1, U702.39 (STEP), U706.1 (1A)
- new net AX1_A1: J711.1 (Pin_1), U701.4 (AOUT1), U701.5 (AOUT1), U701.6 (AOUT1)
- new net AX1_A2: J711.2 (Pin_2), U701.7 (AOUT2), U701.8 (AOUT2), U701.9 (AOUT2)
- new net AX1_B1: J711.3 (Pin_3), U701.17 (BOUT1), U701.18 (BOUT1), U701.19 (BOUT1)
- new net AX1_B2: J711.4 (Pin_4), U701.14 (BOUT2), U701.15 (BOUT2), U701.16 (BOUT2)
- new net AX1_CMD: R761.1, U704.13 (IO1_0), U711.2 (1B)
- new net AX1_CPH: C713.1, U701.44 (CPH)
- new net AX1_CPL: C713.2, U701.43 (CPL)
- new net AX1_CS_N: R713.2, U701.34 (nSCS), U704.9 (IO0_5)
- new net AX1_DIR_INV: U705.6 (3Y), U705.9 (4A)
- new net AX1_DVDD: C716.1, U701.24 (DVDD)
- new net AX1_EXT_DIR_OUT: J701.3 (Pin_3), R753.2
- new net AX1_EXT_DIR_RAW: R753.1, U705.8 (4Y)
- new net AX1_EXT_EN: JP701.3 (Pin_3), R716.1, U705.11 (5A)
- new net AX1_EXT_EN_N_OUT: J701.1 (Pin_1), R751.2
- new net AX1_EXT_EN_N_RAW: R751.1, U705.10 (5Y)
- new net AX1_EXT_STEP_OUT: J701.2 (Pin_2), R752.2
- new net AX1_EXT_STEP_RAW: R752.1, U705.4 (2Y)
- new net AX1_GATED_CMD: JP701.2 (Pin_2), U711.3 (1Y)
- new net AX1_MODE: R715.2, U701.28 (MODE)
- new net AX1_ONBOARD_EN: JP701.1 (Pin_1), R711.1, U701.41 (ENABLE)
- new net AX1_SLEEP_N: R712.2, U701.42 (nSLEEP)
- new net AX1_STEP_INV: U705.2 (1Y), U705.3 (2A)
- new net AX1_VCP: C714.1, U701.1 (VCP)
- new net AX2_A1: J712.1 (Pin_1), U702.4 (AOUT1), U702.5 (AOUT1), U702.6 (AOUT1)
- new net AX2_A2: J712.2 (Pin_2), U702.7 (AOUT2), U702.8 (AOUT2), U702.9 (AOUT2)
- new net AX2_B1: J712.3 (Pin_3), U702.17 (BOUT1), U702.18 (BOUT1), U702.19 (BOUT1)
- new net AX2_B2: J712.4 (Pin_4), U702.14 (BOUT2), U702.15 (BOUT2), U702.16 (BOUT2)
- new net AX2_CMD: R762.1, U704.14 (IO1_1), U711.5 (2B)
- new net AX2_CPH: C723.1, U702.44 (CPH)
- new net AX2_CPL: C723.2, U702.43 (CPL)
- new net AX2_CS_N: R723.2, U702.34 (nSCS), U704.10 (IO0_6)
- new net AX2_DIR_INV: U706.6 (3Y), U706.9 (4A)
- new net AX2_DVDD: C726.1, U702.24 (DVDD)
- new net AX2_EXT_DIR_OUT: J702.3 (Pin_3), R756.2
- new net AX2_EXT_DIR_RAW: R756.1, U706.8 (4Y)
- new net AX2_EXT_EN: JP702.3 (Pin_3), R726.1, U706.11 (5A)
- new net AX2_EXT_EN_N_OUT: J702.1 (Pin_1), R754.2
- new net AX2_EXT_EN_N_RAW: R754.1, U706.10 (5Y)
- new net AX2_EXT_STEP_OUT: J702.2 (Pin_2), R755.2
- new net AX2_EXT_STEP_RAW: R755.1, U706.4 (2Y)
- new net AX2_GATED_CMD: JP702.2 (Pin_2), U711.6 (2Y)
- new net AX2_MODE: R725.2, U702.28 (MODE)
- new net AX2_ONBOARD_EN: JP702.1 (Pin_1), R721.1, U702.41 (ENABLE)
- new net AX2_SLEEP_N: R722.2, U702.42 (nSLEEP)
- new net AX2_STEP_INV: U706.2 (1Y), U706.3 (2A)
- new net AX2_VCP: C724.1, U702.1 (VCP)
- new net AX3_A1: J713.1 (Pin_1), U703.4 (AOUT1), U703.5 (AOUT1), U703.6 (AOUT1)
- new net AX3_A2: J713.2 (Pin_2), U703.7 (AOUT2), U703.8 (AOUT2), U703.9 (AOUT2)
- new net AX3_B1: J713.3 (Pin_3), U703.17 (BOUT1), U703.18 (BOUT1), U703.19 (BOUT1)
- new net AX3_B2: J713.4 (Pin_4), U703.14 (BOUT2), U703.15 (BOUT2), U703.16 (BOUT2)
- new net AX3_CMD: R763.1, U704.15 (IO1_2), U711.10 (3B)
- new net AX3_CPH: C733.1, U703.44 (CPH)
- new net AX3_CPL: C733.2, U703.43 (CPL)
- new net AX3_CS_N: R733.2, U703.34 (nSCS), U704.11 (IO0_7)
- new net AX3_DIR_INV: U707.6 (3Y), U707.9 (4A)
- new net AX3_DVDD: C736.1, U703.24 (DVDD)
- new net AX3_EXT_DIR_OUT: J703.3 (Pin_3), R759.2
- new net AX3_EXT_DIR_RAW: R759.1, U707.8 (4Y)
- new net AX3_EXT_EN: JP703.3 (Pin_3), R736.1, U707.11 (5A)
- new net AX3_EXT_EN_N_OUT: J703.1 (Pin_1), R757.2
- new net AX3_EXT_EN_N_RAW: R757.1, U707.10 (5Y)
- new net AX3_EXT_STEP_OUT: J703.2 (Pin_2), R758.2
- new net AX3_EXT_STEP_RAW: R758.1, U707.4 (2Y)
- new net AX3_GATED_CMD: JP703.2 (Pin_2), U711.8 (3Y)
- new net AX3_MODE: R735.2, U703.28 (MODE)
- new net AX3_ONBOARD_EN: JP703.1 (Pin_1), R731.1, U703.41 (ENABLE)
- new net AX3_SLEEP_N: R732.2, U703.42 (nSLEEP)
- new net AX3_STEP_INV: U707.2 (1Y), U707.3 (2A)
- new net AX3_VCP: C734.1, U703.1 (VCP)
- new net BTN_BACK: U704.4 (IO0_0)
- new net BTN_HOME: U704.6 (IO0_2)
- new net BTN_NEXT: U704.5 (IO0_1)
- new net CPU_ALLOW: U711.11 (4Y), U712.2 (1B), U712.6 (2B)
- new net ESP_EN: U710.3 (EN)
- new net I2C_SCL: U704.22 (SCL)
- new net I2C_SDA: U704.23 (SDA)
- new net IO_INT_N: U704.1 (~{INT})
- new net LED_STAT: U710.6 (WDI)
- new net RLY1_CMD: R764.1, U704.7 (IO0_3), U712.1 (1A)
- new net RLY2_CMD: R765.1, U704.8 (IO0_4), U712.5 (2A)
- new net STEP3_DIR: R738.1, U703.40 (DIR), U707.5 (3A)
- new net STEP3_PUL: R737.1, U703.39 (STEP), U707.1 (1A)
- new net STEP_ARM: R744.1, U708.13 (4B), U709.3 (CLK1), U711.12 (4A)
- new net STEP_ARM_Q: U704.18 (IO1_5), U708.12 (4A), U709.5 (Q1), U711.13 (4B)
- new net STEP_CLEAR_A: U708.3 (1Y), U708.9 (3A)
- new net STEP_CLEAR_B: U708.10 (3B), U708.6 (2Y)
- new net STEP_CLEAR_N: U708.8 (3Y), U709.1 (nCLR1)
- new net STEP_FAULT_N: R714.2, R724.2, R734.2, U701.26 (nFAULT), U702.26 (nFAULT), U703.26 (nFAULT), U704.16 (IO1_3), U708.4 (2A)
- new net STEP_PERMIT: U708.11 (4Y), U711.1 (1A), U711.4 (2A), U711.9 (3A)
- new net STEP_SPI_MISO: R749.1, U701.36 (SDO), U702.36 (SDO), U703.36 (SDO)
- new net STEP_SPI_MOSI: R748.1, U701.37 (SDI), U702.37 (SDI), U703.37 (SDI)
- new net STEP_SPI_SCLK: R747.1, U701.38 (SCLK), U702.38 (SCLK), U703.38 (SCLK)
- new net STEP_WD_CWD: R746.2, U710.2 (CWD)
- new net STEP_WD_OK: R745.2, U704.17 (IO1_4), U708.2 (1B), U710.7 (WDO)
- new net STEP_WD_READY: R750.2, U708.5 (2B), U710.8 (ENOUT)
- new net Z_MAX_IN: U704.20 (IO1_7)
- new net Z_MIN_IN: U704.19 (IO1_6)
- no-connect marks 2 -> 27
Other:
- note added: "2 A RMS normal design target; 3 A RMS NOT thermally qualified. EXT: 5V TTL, EN active LOW. Powered hot-plug not supported."
- note added: "REV 1.2: THREE DRV8462 AXES — HARDWARE ARM / WATCHDOG / EXTERNAL OUTPUTS"
- note removed: "SHEET 4: DUAL STEPSTICK STEPPER CHANNELS & DUAL 5V OMRON G5LE RELAY OUTPUTS"
- moved on the sheet: D501, D502, D503, D504, J505, J506, K501, K502, Q501, Q502, R501, R502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

Commit message: Clear root project DRC findings and preserve explicit Ethernet draft status
Parts:
- J505: footprint TerminalBlock_Phoenix:TerminalBlock_Phoenix_MKDS-1,5-3-5.08_1x03_P5.08mm_Horizontal -> abx-footprints:ABX_J505_TerminalBlock_Phoenix_MKDS-1_5-3-5.08_1x03_P5.08mm_Horizontal
- J506: footprint TerminalBlock_Phoenix:TerminalBlock_Phoenix_MKDS-1,5-3-5.08_1x03_P5.08mm_Horizontal -> abx-footprints:ABX_J506_TerminalBlock_Phoenix_MKDS-1_5-3-5.08_1x03_P5.08mm_Horizontal
Changed lines of the file:
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@@
 			)
 		)
-		(property "Footprint" "TerminalBlock_Phoenix:TerminalBlock_Phoenix_MKDS-1,5-3-5.08_1x03_P5.08mm_Horizontal"
+		(property "Footprint" "abx-footprints:ABX_J505_TerminalBlock_Phoenix_MKDS-1_5-3-5.08_1x03_P5.08mm_Horizontal"
 			(at 200.66 414.02 0)
 			(effects
@@
 			)
 		)
-		(property "Footprint" "TerminalBlock_Phoenix:TerminalBlock_Phoenix_MKDS-1,5-3-5.08_1x03_P5.08mm_Horizontal"
+		(property "Footprint" "abx-footprints:ABX_J506_TerminalBlock_Phoenix_MKDS-1_5-3-5.08_1x03_P5.08mm_Horizontal"
 			(at 383.54 414.02 0)
 			(effects
