File: variants/ABX-Motion-ETH/abx-motion-eth-placement.kicad_pcb (KiCad board)
At the start: 4 copper layers, 157 x 105 mm, 387 parts, among them J1 XT60_BAT, J102 E_STOP, J201 USB-C, J202 ENC1_CONN, J203 ENC2_CONN, J204 CAN_TERM, J205 CAN_BUS, J206 RS485_TERM, J207 RS485_BUS, J208 OLED_I2C, J209 I2C_EXP, J301 MOTOR_OUT, J401 MOTOR_OUT, J505 RELAY1_OUT, J506 RELAY2_OUT, J601 B3B-PH-K-S, J602 B3B-PH-K-S, J603 B3B-PH-K-S, J604 B3B-PH-K-S, J605 B3B-PH-K-S, J606 B3B-PH-K-S, J607 B3B-PH-K-S, J608 B3B-PH-K-S, J701 EXT 5V TTL EN_N STEP DIR GND, J702 EXT 5V TTL EN_N STEP DIR GND, J703 EXT 5V TTL EN_N STEP DIR GND, J711 JST-XH MOTOR 1, J712 JST-XH MOTOR 2, J713 JST-XH MOTOR 3, J801 HR911105A / C12074, K501 G5LE-14-DC5, K502 G5LE-14-DC5, Q1 SQJ459EP-T1_GE3, Q301 CSD18540Q5B, Q302 CSD18540Q5B, Q303 CSD18540Q5B, Q304 CSD18540Q5B, Q401 CSD18540Q5B, Q402 CSD18540Q5B, Q403 CSD18540Q5B, Q404 CSD18540Q5B, Q501 AO3400A, Q502 AO3400A, Q601 AO3400A, Q602 AO3400A, Q801 RESET SINK / SELECT, SW201 RESET, SW202 BOOT, SW203 BTN_BACK, SW204 BTN_NEXT, SW205 BTN_HOME, U1 LMR36520FADDA, U2 AP2112K-3.3, U201 USBLC6-2SC6, U202 TCAN1042V-Q1, U203 THVD1450DR, U3 ESP32-S3-WROOM-1-N8R2, U301 DRV8701ERGER, U4 74LVC14A, U401 DRV8701ERGER, U601 PCA9555PW,118, U701 DRV8462DDWR, U702 DRV8462DDWR, U703 DRV8462DDWR, U704 PCA9555PW,118, U705 SN74AHCT14PWR, U706 SN74AHCT14PWR, U707 SN74AHCT14PWR, U708 SN74HC08PWR, U709 SN74HC74PWR, U710 TPS3431SDRBR, U711 SN74HC08PWR, U712 SN74LVC2G08DCUR, U801 W5500 / C32843, U803 OPEN-DRAIN RESET / SELECT, Y801 25MHz / CL TO SELECT

Commit message: Move Ethernet draft CS test pads to left of ESP32
Parts:
- moved TP_CS1 50.3 mm to (82.5, 51.0), turned to 90 degrees
- moved TP_CS2 49.3 mm to (88.0, 51.0), turned to 90 degrees
Changed lines of the file:
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@@
 	(footprint "TestPoint:TestPoint_Pad_D1.5mm"
 		(layer "F.Cu")
-		(at 137 56.5)
+		(at 88 51 90)
 		(descr "SMD pad as test Point, diameter 1.5mm")
 		(tags "test point SMD pad")
 		(property "Reference" "TP_CS2"
-			(at 0 -1.648 0)
+			(at 0 -1.648 90)
 			(layer "F.Fab")
 			(hide yes)
@@
 		)
 		(property "Value" "TP_CS"
-			(at 0 1.75 0)
+			(at 0 1.75 90)
 			(layer "F.Fab")
 			(hide yes)
@@
 		)
 		(property "Datasheet" ""
-			(at 0 0 0)
+			(at 0 0 90)
 			(unlocked yes)
 			(layer "F.Fab")
@@
 		)
 		(property "Description" ""
-			(at 0 0 0)
+			(at 0 0 90)
 			(unlocked yes)
 			(layer "F.Fab")
@@
 		(duplicate_pad_numbers_are_jumpers no)
 		(fp_line
-			(start -1.4 -1.9)
-			(end 1.4 -1.9)
+			(start 1.4 -1.9)
+			(end 1.4 1.9)
 			(stroke
 				(width 0.05)
@@
 		)
 		(fp_line
-			(start -1.4 1.9)
-			(end -1.4 -1.9)
+			(start -1.4 -1.9)
+			(end 1.4 -1.9)
 			(stroke
 				(width 0.05)
@@
 		)
 		(fp_line
-			(start 1.4 -1.9)
-			(end 1.4 1.9)
+			(start 1.4 1.9)
+			(end -1.4 1.9)
 			(stroke
 				(width 0.05)
@@
 		)
 		(fp_line
-			(start 1.4 1.9)
-			(end -1.4 1.9)
+			(start -1.4 1.9)
+			(end -1.4 -1.9)
 			(stroke
 				(width 0.05)
@@
 		)
 		(fp_line
-			(start -1.4 -1.9)
-			(end 1.4 -1.9)
+			(start 1.4 -1.9)
+			(end 1.4 1.9)
 			(stroke
 				(width 0.05)
@@
 		)
 		(fp_line
-			(start -1.4 1.9)
-			(end -1.4 -1.9)
+			(start -1.4 -1.9)
+			(end 1.4 -1.9)
 			(stroke
 				(width 0.05)
@@
 		)
 		(fp_line
-			(start 1.4 -1.9)
-			(end 1.4 1.9)
+			(start 1.4 1.9)
+			(end -1.4 1.9)
 			(stroke
 				(width 0.05)
@@
 		)
 		(fp_line
-			(start 1.4 1.9)
-			(end -1.4 1.9)
+			(start -1.4 1.9)
+			(end -1.4 -1.9)
 			(stroke
 				(width 0.05)
@@
 		)
 		(pad "1" thru_hole roundrect
-			(at 0 0)
+			(at 0 0 90)
 			(size 2.5 3.6)
 			(drill 1)
@@
 	(footprint "TestPoint:TestPoint_Pad_D1.5mm"
 		(layer "F.Cu")
-		(at 132.5 56.5)
+		(at 82.5 51 90)
 		(descr "SMD pad as test Point, diameter 1.5mm")
 		(tags "test point SMD pad")
 		(property "Reference" "TP_CS1"
-			(at 0 -1.648 0)
+			(at 0 -1.648 90)
 			(layer "F.Fab")
 			(hide yes)
@@
 		)
 		(property "Value" "TP_CS"
-			(at 0 1.75 0)
+			(at 0 1.75 90)
 			(layer "F.Fab")
 			(hide yes)
@@
 		)
 		(property "Datasheet" ""
-			(at 0 0 0)
+			(at 0 0 90)
 			(unlocked yes)
 			(layer "F.Fab")
@@
 		)
 		(property "Description" ""
-			(at 0 0 0)
+			(at 0 0 90)
 			(unlocked yes)
 			(layer "F.Fab")
@@
 		(duplicate_pad_numbers_are_jumpers no)
 		(fp_line
-			(start -1.4 -1.9)
-			(end 1.4 -1.9)
+			(start 1.4 -1.9)
+			(end 1.4 1.9)
 			(stroke
 				(width 0.05)
@@
 		)
 		(fp_line
-			(start -1.4 1.9)
-			(end -1.4 -1.9)
+			(start -1.4 -1.9)
+			(end 1.4 -1.9)
 			(stroke
 				(width 0.05)
@@
 		)
 		(fp_line
-			(start 1.4 -1.9)
-			(end 1.4 1.9)
+			(start 1.4 1.9)
+			(end -1.4 1.9)
 			(stroke
 				(width 0.05)
@@
 		)
 		(fp_line
-			(start 1.4 1.9)
-			(end -1.4 1.9)
+			(start -1.4 1.9)
+			(end -1.4 -1.9)
 			(stroke
 				(width 0.05)
@@
 		)
 		(fp_line
-			(start -1.4 -1.9)
-			(end 1.4 -1.9)
+			(start 1.4 -1.9)
+			(end 1.4 1.9)
 			(stroke
 				(width 0.05)
@@
 		)
 		(fp_line
-			(start -1.4 1.9)
-			(end -1.4 -1.9)
+			(start -1.4 -1.9)
+			(end 1.4 -1.9)
 			(stroke
 				(width 0.05)
@@
 		)
 		(fp_line
-			(start 1.4 -1.9)
-			(end 1.4 1.9)
+			(start 1.4 1.9)
+			(end -1.4 1.9)
 			(stroke
 				(width 0.05)
@@
 		)
 		(fp_line
-			(start 1.4 1.9)
-			(end -1.4 1.9)
+			(start -1.4 1.9)
+			(end -1.4 -1.9)
 			(stroke
 				(width 0.05)
@@
 		)
 		(pad "1" thru_hole roundrect
-			(at 0 0)
+			(at 0 0 90)
 			(size 2.5 3.6)
 			(drill 1)
@@
 	)
 	(gr_text "CS1"
-		(at 132.5 53.65 0)
+		(at 82.5 48.55 0)
 		(layer "F.SilkS")
 		(effects
@@
 	)
 	(gr_text "CS2"
-		(at 137 53.65 0)
+		(at 88 48.55 0)
 		(layer "F.SilkS")
 		(effects
@@
 	)
 	(gr_text "CS1"
-		(at 132.5 53.65 0)
+		(at 82.5 48.55 0)
 		(layer "B.SilkS")
 		(effects
@@
 	)
 	(gr_text "CS2"
-		(at 137 53.65 0)
+		(at 88 48.55 0)
 		(layer "B.SilkS")
 		(effects
