File: variants/ABX-Motion-ETH/abx-motion-eth-placement.kicad_pcb (KiCad board)
At the start: 4 copper layers, 157 x 105 mm, 387 parts, among them J1 XT60_BAT, J102 E_STOP, J201 USB-C, J202 ENC1_CONN, J203 ENC2_CONN, J204 CAN_TERM, J205 CAN_BUS, J206 RS485_TERM, J207 RS485_BUS, J208 OLED_I2C, J209 I2C_EXP, J301 MOTOR_OUT, J401 MOTOR_OUT, J505 RELAY1_OUT, J506 RELAY2_OUT, J601 B3B-PH-K-S, J602 B3B-PH-K-S, J603 B3B-PH-K-S, J604 B3B-PH-K-S, J605 B3B-PH-K-S, J606 B3B-PH-K-S, J607 B3B-PH-K-S, J608 B3B-PH-K-S, J701 EXT 5V TTL EN_N STEP DIR GND, J702 EXT 5V TTL EN_N STEP DIR GND, J703 EXT 5V TTL EN_N STEP DIR GND, J711 JST-XH MOTOR 1, J712 JST-XH MOTOR 2, J713 JST-XH MOTOR 3, J801 HR911105A / C12074, K501 G5LE-14-DC5, K502 G5LE-14-DC5, Q1 SQJ459EP-T1_GE3, Q301 CSD18540Q5B, Q302 CSD18540Q5B, Q303 CSD18540Q5B, Q304 CSD18540Q5B, Q401 CSD18540Q5B, Q402 CSD18540Q5B, Q403 CSD18540Q5B, Q404 CSD18540Q5B, Q501 AO3400A, Q502 AO3400A, Q601 AO3400A, Q602 AO3400A, Q801 RESET SINK / SELECT, SW201 RESET, SW202 BOOT, SW203 BTN_BACK, SW204 BTN_NEXT, SW205 BTN_HOME, U1 LMR36520FADDA, U2 AP2112K-3.3, U201 USBLC6-2SC6, U202 TCAN1042V-Q1, U203 THVD1450DR, U3 ESP32-S3-WROOM-1-N8R2, U301 DRV8701ERGER, U4 74LVC14A, U401 DRV8701ERGER, U601 PCA9555PW,118, U701 DRV8462DDWR, U702 DRV8462DDWR, U703 DRV8462DDWR, U704 PCA9555PW,118, U705 SN74AHCT14PWR, U706 SN74AHCT14PWR, U707 SN74AHCT14PWR, U708 SN74HC08PWR, U709 SN74HC74PWR, U710 TPS3431SDRBR, U711 SN74HC08PWR, U712 SN74LVC2G08DCUR, U801 W5500 / C32843, U803 OPEN-DRAIN RESET / SELECT, Y801 25MHz / CL TO SELECT

Commit message: Expand Ethernet supply reservation and add draft 3V3 test pad
Parts:
- added TP_ETH_3V3: 3V3_ETH / UNCONNECTED DRAFT, TestPoint:TestPoint_Pad_D1.5mm, F.Cu at (133.5, 56.2)
- moved PWR_ETH_RESERVE 4.25 mm to (143.5, 56.2)
Other:
- board text added: "3V3_ETH"
Changed lines of the file:
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@@
 	(footprint ""
 		(layer "F.Cu")
-		(at 147.75 56.25)
+		(at 143.5 56.25)
 		(property "Reference" "PWR_ETH_RESERVE"
 			(at 0 0 0)
@@
 		(duplicate_pad_numbers_are_jumpers no)
 		(fp_line
-			(start -8.25 -2.25)
-			(end 8.25 -2.25)
-			(stroke
-				(width 0.15)
-				(type default)
-			)
-			(layer "Dwgs.User")
-		)
-		(fp_line
-			(start -8.25 2.25)
-			(end -8.25 -2.25)
-			(stroke
-				(width 0.15)
-				(type default)
-			)
-			(layer "Dwgs.User")
-		)
-		(fp_line
-			(start 8.25 -2.25)
-			(end 8.25 2.25)
-			(stroke
-				(width 0.15)
-				(type default)
-			)
-			(layer "Dwgs.User")
-		)
-		(fp_line
-			(start 8.25 2.25)
-			(end -8.25 2.25)
+			(start -12.5 -2.25)
+			(end 12.5 -2.25)
+			(stroke
+				(width 0.15)
+				(type default)
+			)
+			(layer "Dwgs.User")
+		)
+		(fp_line
+			(start -12.5 2.25)
+			(end -12.5 -2.25)
+			(stroke
+				(width 0.15)
+				(type default)
+			)
+			(layer "Dwgs.User")
+		)
+		(fp_line
+			(start 12.5 -2.25)
+			(end 12.5 2.25)
+			(stroke
+				(width 0.15)
+				(type default)
+			)
+			(layer "Dwgs.User")
+		)
+		(fp_line
+			(start 12.5 2.25)
+			(end -12.5 2.25)
 			(stroke
 				(width 0.15)
@@
 				(thickness 0.12)
 			)
+		)
+	)
+	(footprint "TestPoint:TestPoint_Pad_D1.5mm"
+		(layer "F.Cu")
+		(at 133.5 56.25)
+		(descr "SMD pad as test Point, diameter 1.5mm")
+		(tags "test point SMD pad")
+		(property "Reference" "TP_ETH_3V3"
+			(at 0 -1.648 0)
+			(layer "F.SilkS")
+			(hide yes)
+			(effects
+				(font
+					(size 1 1)
+					(thickness 0.15)
+				)
+			)
+		)
+		(property "Value" "3V3_ETH / UNCONNECTED DRAFT"
+			(at 0 1.75 0)
+			(layer "F.Fab")
+			(hide yes)
+			(effects
+				(font
+					(size 1 1)
+					(thickness 0.15)
+				)
+			)
+		)
+		(property "Datasheet" ""
+			(at 0 0 0)
+			(unlocked yes)
+			(layer "F.Fab")
+			(hide yes)
+			(effects
+				(font
+					(size 1.27 1.27)
+					(thickness 0.15)
+				)
+			)
+		)
+		(property "Description" ""
+			(at 0 0 0)
+			(unlocked yes)
+			(layer "F.Fab")
+			(hide yes)
+			(effects
+				(font
+					(size 1.27 1.27)
+					(thickness 0.15)
+				)
+			)
+		)
+		(attr exclude_from_pos_files exclude_from_bom)
+		(duplicate_pad_numbers_are_jumpers no)
+		(fp_circle
+			(center 0 0)
+			(end 0 0.95)
+			(stroke
+				(width 0.12)
+				(type solid)
+			)
+			(fill no)
+			(layer "F.SilkS")
+		)
+		(fp_circle
+			(center 0 0)
+			(end 1.25 0)
+			(stroke
+				(width 0.05)
+				(type solid)
+			)
+			(fill no)
+			(layer "F.CrtYd")
+		)
+		(fp_text user "${REFERENCE}"
+			(at 0 -1.65 0)
+			(layer "F.Fab")
+			(effects
+				(font
+					(size 1 1)
+					(thickness 0.15)
+				)
+			)
+		)
+		(pad "1" smd circle
+			(at 0 0)
+			(size 1.5 1.5)
+			(layers "F.Cu" "F.Mask")
+		)
+		(embedded_fonts no)
+	)
+	(gr_text "3V3_ETH"
+		(at 133.5 54.4 0)
+		(layer "F.SilkS")
+		(effects
+			(font
+				(size 0.65 0.65)
+				(thickness 0.12)
+			)
