File: variants/ABX-Motion-ETH/abx-motion-eth-placement.kicad_pcb (KiCad board)
At the start: 4 copper layers, 157 x 105 mm, 405 parts, among them J1 XT60_BAT, J102 E_STOP, J201 USB-C, J202 ENC1_CONN, J203 ENC2_CONN, J204 CAN_TERM, J205 CAN_BUS, J206 RS485_TERM, J207 RS485_BUS, J208 OLED_I2C, J209 I2C_EXP, J301 MOTOR_OUT, J401 MOTOR_OUT, J505 RELAY1_OUT, J506 RELAY2_OUT, J601 B3B-PH-K-S, J602 B3B-PH-K-S, J603 B3B-PH-K-S, J604 B3B-PH-K-S, J605 B3B-PH-K-S, J606 B3B-PH-K-S, J607 B3B-PH-K-S, J608 B3B-PH-K-S, J701 EXT 5V TTL EN_N STEP DIR GND, J702 EXT 5V TTL EN_N STEP DIR GND, J703 EXT 5V TTL EN_N STEP DIR GND, J711 JST-XH MOTOR 1, J712 JST-XH MOTOR 2, J713 JST-XH MOTOR 3, J801 HR911105A / C12074, K501 G5LE-14-DC5, K502 G5LE-14-DC5, Q1 SQJ459EP-T1_GE3, Q301 CSD18540Q5B, Q302 CSD18540Q5B, Q303 CSD18540Q5B, Q304 CSD18540Q5B, Q401 CSD18540Q5B, Q402 CSD18540Q5B, Q403 CSD18540Q5B, Q404 CSD18540Q5B, Q501 AO3400A, Q502 AO3400A, Q601 AO3400A, Q602 AO3400A, Q801 BSS138, Q802 BSS138, SW201 RESET, SW202 BOOT, SW203 BTN_BACK, SW204 BTN_NEXT, SW205 BTN_HOME, U1 LMR36520FADDA, U2 AP2112K-3.3, U201 USBLC6-2SC6, U202 TCAN1042V-Q1, U203 THVD1450DR, U3 ESP32-S3-WROOM-1-N8R2, U301 DRV8701ERGER, U4 74LVC14A, U401 DRV8701ERGER, U601 PCA9555PW,118, U701 DRV8462DDWR, U702 DRV8462DDWR, U703 DRV8462DDWR, U704 PCA9555PW,118, U705 SN74AHCT14PWR, U706 SN74AHCT14PWR, U707 SN74AHCT14PWR, U708 SN74HC08PWR, U709 SN74HC74PWR, U710 TPS3431SDRBR, U711 SN74HC08PWR, U712 SN74LVC2G08DCUR, U801 W5500 / C32843, U802 LMR36506R3RPER, U803 TPS3808G33DBVR, U804 TXU0304PWR, Y801 25MHz / CL TO SELECT

Commit message: Begin Rev 1.2b Ethernet routing and clean displaced copper
Parts:
- TP_ETH_3V3: value 3V3_ETH / UNCONNECTED DRAFT -> 3V3_ETH / POWER TEST POINT
Connections:
- C821 pad 1: (no net) -> +BATT
- C821 pad 2: (no net) -> GND
- C822 pad 1: (no net) -> +BATT
- C822 pad 2: (no net) -> GND
- C823 pad 1: (no net) -> GND
- C823 pad 2: (no net) -> +BATT
- C824 pad 1: (no net) -> ETH_BOOT
- C824 pad 2: (no net) -> ETH_SW
- C825 pad 1: (no net) -> ETH_VCC_INT
- C825 pad 2: (no net) -> GND
- C826 pad 1: (no net) -> GND
- C826 pad 2: (no net) -> 3V3_ETH
- C827 pad 1: (no net) -> GND
- C827 pad 2: (no net) -> 3V3_ETH
- L801 pad 1: (no net) -> 3V3_ETH
- L801 pad 2: (no net) -> ETH_SW
- R817 pad 1: (no net) -> +3V3
- R817 pad 2: (no net) -> ETH_BUCK_EN
- R818 pad 1: (no net) -> ETH_BUCK_EN
- R818 pad 2: (no net) -> GND
- TP_ETH_3V3 pad 1: (no net) -> 3V3_ETH
- U802 pad 1: (no net) -> ETH_VCC_INT
- U802 pad 2: (no net) -> unconnected-(U802-PG-Pad2)
- U802 pad 3: (no net) -> ETH_BUCK_EN
- U802 pad 4: (no net) -> +BATT
- U802 pad 5: (no net) -> ETH_SW
- U802 pad 6: (no net) -> ETH_BOOT
- U802 pad 7: (no net) -> ETH_VCC_INT
- U802 pad 8: (no net) -> 3V3_ETH
- U802 pad 9: (no net) -> GND
Routing:
- net 3V3_ETH: track 0.00 -> 43.0 mm, vias 0 -> 3
- net +3V3: track 579.5 -> 610.2 mm, vias 82 -> 81
- net I2C_SDA: track 173.7 -> 154.0 mm
- net GND: track 303.0 -> 321.2 mm, vias 294 -> 295
- net STEP_SPI_SCLK: track 140.0 -> 156.7 mm, vias 9 -> 11
- net +BATT: track 287.8 -> 301.9 mm, vias 75 -> 78
- net +5V: track 316.2 -> 302.8 mm, vias 41 -> 36
- net /M2_CS: track 145.7 -> 133.6 mm, vias 5 -> 8
- net STEP_SPI_MOSI: track 122.9 -> 133.6 mm, vias 11 -> 13
- net AX1_EXT_EN: track 42.2 -> 32.4 mm, vias 3 -> 7
- net RLY1_CMD: track 55.5 -> 65.0 mm, vias 9 -> 10
- net STEP2_DIR: track 132.5 -> 141.8 mm, vias 11 -> 12
- net STEP_WD_OK: track 76.3 -> 85.1 mm, vias 7 -> 13
- net /M1_PWM_PH: track 128.9 -> 137.5 mm, vias 5 -> 7
- net STEP_SPI_MISO: track 152.3 -> 160.6 mm, vias 14 -> 15
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